File: Hardware/pcb.brd (EAGLE design)
At the start: 170.4 x 111.7 mm, 103 parts, among them IC1 XC6220A331MR-G, IC2 BD5229G-TR, J1 112A-TAAR-R03_ATTEND, J2 QWIIC_RIGHT_ANGLE, J3 FH34SRJ-24S-0.5SH_99_, J4 SAMACSYS_PARTS_USB4110-GF-A, Q1 20V/4.2A/52mΩ/1.4W, Q2 SI1308EDL-T1-GE3, Q3 20V/4.2A/52mΩ/1.4W, U1 MAX17048G+T10, U2 W25Q512JVEIQ, U3 ESP32-C6-WROOM-1-N8, U4 ESP32_WROVER_BME680_BME680, U5 DS3231SN#

Commit message: Am realizat ca nu am copiat repo-ul deloc
Am aliniat butoanele, si am completat issue-urile
Parts:
- moved R19 3.45 mm to (58.1, 108.6)
- moved C2 2.78 mm to (172.4, 14.1)
- moved C9 2.61 mm to (12.1, 99.2)
- moved C21 2.04 mm to (51.8, 108.4)
- moved C24 1.38 mm to (66.6, 108.6)
- moved R21 1.09 mm to (26.9, 109.3)
- moved U$2 0.74 mm to (54.8, 109.2)
- moved U$1 0.66 mm to (69.9, 109.2)
- moved C23 0.61 mm to (33.8, 108.4)
- moved C22 0.44 mm to (73.3, 108.9)
Routing:
- net 3V3: track 567.9 -> 572.5 mm
- net IO/CHANGE: track 81.3 -> 85.2 mm
- net 12C_PW: track 182.6 -> 184.9 mm
- net GND: track 746.1 -> 748.1 mm
- net N$7: track 15.4 -> 17.1 mm
- net IO/BOOT: track 65.7 -> 64.1 mm
- net SDA: track 224.0 -> 224.5 mm
